File: kicad/control.sch (KiCad schematic (older format))
At the start: 30 parts, among them P2 SWD, Q2 MMBT3904, U3 STM32L052CxTx, U4 MMA8652FC, Y1 32.767KHz

Commit message: Added footprints for most major components
We are missing almost all passives
Parts:
- SP1: footprint (none) -> simple-led-watch:CSS-0575A-SMT
- U4: footprint (none) -> simple-led-watch:10-DFN; Part No. (none) -> MMA8652FCR1CT-ND
- Y1: footprint (none) -> simple-led-watch:XTAL-CPFB; Part No. (none) -> 370-1057-1-ND
Changed lines of the file:
@@
 $EndComp
 $Comp
-L +3.3V #PWR17
+L +3.3V #PWR017
 U 1 1 57FCBB0F
 P 700 700
-F 0 "#PWR17" H 700 550 50  0001 C CNN
+F 0 "#PWR017" H 700 550 50  0001 C CNN
 F 1 "+3.3V" H 700 840 50  0000 C CNN
 F 2 "" H 700 700 50  0000 C CNN
@@
 $EndComp
 $Comp
-L GND #PWR18
+L GND #PWR018
 U 1 1 57FCBBFF
 P 1100 1600
-F 0 "#PWR18" H 1100 1350 50  0001 C CNN
+F 0 "#PWR018" H 1100 1350 50  0001 C CNN
 F 1 "GND" H 1100 1450 50  0000 C CNN
 F 2 "" H 1100 1600 50  0000 C CNN
@@
 $EndComp
 $Comp
-L GND #PWR19
+L GND #PWR019
 U 1 1 57FCBD25
 P 2800 2000
-F 0 "#PWR19" H 2800 1750 50  0001 C CNN
+F 0 "#PWR019" H 2800 1750 50  0001 C CNN
 F 1 "GND" H 2800 1850 50  0000 C CNN
 F 2 "" H 2800 2000 50  0000 C CNN
@@
 $EndComp
 $Comp
-L GND #PWR20
+L GND #PWR020
 U 1 1 57FCBED2
 P 1100 2700
-F 0 "#PWR20" H 1100 2450 50  0001 C CNN
+F 0 "#PWR020" H 1100 2450 50  0001 C CNN
 F 1 "GND" H 1100 2550 50  0000 C CNN
 F 2 "" H 1100 2700 50  0000 C CNN
@@
 F 0 "Y1" H 1300 3400 50  0000 C CNN
 F 1 "32.767KHz" H 1300 3100 50  0000 C CNN
-F 2 "" H 1300 3250 50  0000 C CNN
+F 2 "simple-led-watch:XTAL-CPFB" H 1300 3250 50  0000 C CNN
 F 3 "" H 1300 3250 50  0000 C CNN
+F 4 "370-1057-1-ND" H 1300 3250 60  0001 C CNN "Part No."
 	1    1300 3250
 	0    1    1    0
@@
 $EndComp
 $Comp
-L GND #PWR22
+L GND #PWR021
 U 1 1 57FCC8BD
 P 700 3600
-F 0 "#PWR22" H 700 3350 50  0001 C CNN
+F 0 "#PWR021" H 700 3350 50  0001 C CNN
 F 1 "GND" H 700 3450 50  0000 C CNN
 F 2 "" H 700 3600 50  0000 C CNN
@@
 $EndComp
 $Comp
-L GND #PWR25
+L GND #PWR022
 U 1 1 5801A8C3
 P 1500 5000
-F 0 "#PWR25" H 1500 4750 50  0001 C CNN
+F 0 "#PWR022" H 1500 4750 50  0001 C CNN
 F 1 "GND" H 1500 4850 50  0000 C CNN
 F 2 "" H 1500 5000 50  0000 C CNN
@@
 STM32_RESET
 $Comp
-L GND #PWR23
+L GND #PWR023
 U 1 1 5801ADFC
 P 2800 4200
-F 0 "#PWR23" H 2800 3950 50  0001 C CNN
+F 0 "#PWR023" H 2800 3950 50  0001 C CNN
 F 1 "GND" H 2800 4050 50  0000 C CNN
 F 2 "" H 2800 4200 50  0000 C CNN
@@
 F 0 "U4" H 2400 6050 50  0000 C CNN
 F 1 "MMA8652FC" H 2400 7050 50  0000 C CNN
-F 2 "" H 2400 6500 50  0001 C CNN
+F 2 "simple-led-watch:10-DFN" H 2400 6500 50  0001 C CNN
 F 3 "" H 2400 6500 50  0001 C CNN
+F 4 "MMA8652FCR1CT-ND" H 2400 6500 60  0001 C CNN "Part No."
 	1    2400 6500
 	1    0    0    -1
@@
 $EndComp
 $Comp
-L +3.3V #PWR26
+L +3.3V #PWR024
 U 1 1 5801C871
 P 700 5400
-F 0 "#PWR26" H 700 5250 50  0001 C CNN
+F 0 "#PWR024" H 700 5250 50  0001 C CNN
 F 1 "+3.3V" H 700 5540 50  0000 C CNN
 F 2 "" H 700 5400 50  0000 C CNN
@@
 $EndComp
 $Comp
-L GND #PWR30
+L GND #PWR025
 U 1 1 5801C913
 P 700 6800
-F 0 "#PWR30" H 700 6550 50  0001 C CNN
+F 0 "#PWR025" H 700 6550 50  0001 C CNN
 F 1 "GND" H 700 6650 50  0000 C CNN
 F 2 "" H 700 6800 50  0000 C CNN
@@
 $EndComp
 $Comp
-L GND #PWR31
+L GND #PWR026
 U 1 1 5801CB03
 P 1800 6900
-F 0 "#PWR31" H 1800 6650 50  0001 C CNN
+F 0 "#PWR026" H 1800 6650 50  0001 C CNN
 F 1 "GND" H 1800 6750 50  0000 C CNN
 F 2 "" H 1800 6900 50  0000 C CNN
@@
 $EndComp
 $Comp
-L GND #PWR32
+L GND #PWR027
 U 1 1 5801CE9C
 P 1500 7300
-F 0 "#PWR32" H 1500 7050 50  0001 C CNN
+F 0 "#PWR027" H 1500 7050 50  0001 C CNN
 F 1 "GND" H 1500 7150 50  0000 C CNN
 F 2 "" H 1500 7300 50  0000 C CNN
@@
 $EndComp
 $Comp
-L +3.3V #PWR27
+L +3.3V #PWR028
 U 1 1 5801D568
 P 8900 5400
-F 0 "#PWR27" H 8900 5250 50  0001 C CNN
+F 0 "#PWR028" H 8900 5250 50  0001 C CNN
 F 1 "+3.3V" H 8900 5540 50  0000 C CNN
 F 2 "" H 8900 5400 50  0000 C CNN
@@
 $EndComp
 $Comp
-L +3.3V #PWR28
+L +3.3V #PWR029
 U 1 1 5801E31A
 P 3000 5600
-F 0 "#PWR28" H 3000 5450 50  0001 C CNN
+F 0 "#PWR029" H 3000 5450 50  0001 C CNN
 F 1 "+3.3V" H 3000 5740 50  0000 C CNN
 F 2 "" H 3000 5600 50  0000 C CNN
@@
 Connection ~ 9000 3300
 $Comp
-L +3.3V #PWR21
+L +3.3V #PWR030
 U 1 1 5801C3D8
 P 9000 2800
-F 0 "#PWR21" H 9000 2650 50  0001 C CNN
+F 0 "#PWR030" H 9000 2650 50  0001 C CNN
 F 1 "+3.3V" H 9000 2940 50  0000 C CNN
 F 2 "" H 9000 2800 50  0000 C CNN
@@
 F 0 "SP1" H 7200 5450 50  0000 C CNN
 F 1 "CSS-0575A-SMT" H 7200 4950 50  0000 C CNN
-F 2 "" H 7300 5200 50  0000 C CNN
+F 2 "simple-led-watch:CSS-0575A-SMT" H 7300 5200 50  0001 C CNN
 F 3 "" H 7300 5200 50  0000 C CNN
 F 4 "102-2201-1-ND" H 7300 5200 60  0001 C CNN "Part No."
@@
 $EndComp
 $Comp
-L +3.3V #PWR24
+L +3.3V #PWR031
 U 1 1 58024910
 P 6700 4850
-F 0 "#PWR24" H 6700 4700 50  0001 C CNN
+F 0 "#PWR031" H 6700 4700 50  0001 C CNN
 F 1 "+3.3V" H 6700 4990 50  0000 C CNN
 F 2 "" H 6700 4850 50  0000 C CNN
@@
 	6200 6100 6400 6100
 $Comp
-L GND #PWR29
+L GND #PWR032
 U 1 1 58024E53
 P 6700 6400
-F 0 "#PWR29" H 6700 6150 50  0001 C CNN
+F 0 "#PWR032" H 6700 6150 50  0001 C CNN
 F 1 "GND" H 6700 6250 50  0000 C CNN
 F 2 "" H 6700 6400 50  0000 C CNN

Commit message: Completed initial placement of major components
The passives are causing trouble. We need to eliminate every pullup
possible.
Parts:
- C10, C12, C16, C17, C18, C8, C9: footprint (none) -> Capacitors_SMD:C_0402; Part No. (none) -> 1276-1022-1-ND
- C11, C15: footprint (none) -> Capacitors_SMD:C_0402; Part No. (none) -> 1276-1448-1-ND
- C13, C14: footprint (none) -> Capacitors_SMD:C_0402
- C7: footprint (none) -> Capacitors_SMD:C_0402; Part No. (none) -> 1276-6830-1-ND
- D4: value D_Small -> RB521S30T5G; footprint (none) -> Diodes_SMD:SOD-523; Part No. (none) -> B521S30T5GOSCT-ND
- L2: footprint (none) -> Resistors_SMD:R_0603; Part No. (none) -> 445-6755-1-ND
- R10, R11, R12, R13, R14, R15, R16, R17, R18, R9: footprint (none) -> Resistors_SMD:R_0402
Connections:
- net ACCEL_VDD is gone; now on net +3V3: C15.1, C16.1, C17.1, R14.2, U4.1 (VDD), U4.8 (VDDIO)
- net STM32_VDD is gone; now on net +3V3: C10.1, C7.1, C8.1, C9.1, L2.2, R9.2, U3.1 (VDD), U3.24 (VDD), U3.36 (VDD_USB), U3.48 (VDD)
- net USB_D+_R renamed USB_D_R+
- net USB_D-_R renamed USB_D_R-
Changed lines of the file:
@@
 F 0 "C8" H 1425 1350 50  0000 L CNN
 F 1 "0.1u" H 1425 1150 50  0000 L CNN
-F 2 "" H 1438 1100 50  0000 C CNN
+F 2 "Capacitors_SMD:C_0402" H 1438 1100 50  0001 C CNN
 F 3 "" H 1400 1250 50  0000 C CNN
+F 4 "1276-1022-1-ND" H 1400 1250 60  0001 C CNN "Part No."
 	1    1400 1250
 	1    0    0    -1
@@
 F 0 "C9" H 1725 1350 50  0000 L CNN
 F 1 "0.1u" H 1725 1150 50  0000 L CNN
-F 2 "" H 1738 1100 50  0000 C CNN
+F 2 "Capacitors_SMD:C_0402" H 1738 1100 50  0001 C CNN
 F 3 "" H 1700 1250 50  0000 C CNN
+F 4 "1276-1022-1-ND" H 1700 1250 60  0001 C CNN "Part No."
 	1    1700 1250
 	1    0    0    -1
@@
 F 0 "C10" H 2025 1350 50  0000 L CNN
 F 1 "0.1u" H 2025 1150 50  0000 L CNN
-F 2 "" H 2038 1100 50  0000 C CNN
+F 2 "Capacitors_SMD:C_0402" H 2038 1100 50  0001 C CNN
 F 3 "" H 2000 1250 50  0000 C CNN
+F 4 "1276-1022-1-ND" H 2000 1250 60  0001 C CNN "Part No."
 	1    2000 1250
 	1    0    0    -1
@@
 F 0 "C7" H 1125 1350 50  0000 L CNN
 F 1 "10u" H 1125 1150 50  0000 L CNN
-F 2 "" H 1138 1100 50  0000 C CNN
+F 2 "Capacitors_SMD:C_0402" H 1138 1100 50  0001 C CNN
 F 3 "" H 1100 1250 50  0000 C CNN
+F 4 "1276-6830-1-ND" H 1100 1250 60  0001 C CNN "Part No."
 	1    1100 1250
 	1    0    0    -1
@@
 F 0 "C12" H 1425 2450 50  0000 L CNN
 F 1 "0.1u" H 1425 2250 50  0000 L CNN
-F 2 "" H 1438 2200 50  0000 C CNN
+F 2 "Capacitors_SMD:C_0402" H 1438 2200 50  0001 C CNN
 F 3 "" H 1400 2350 50  0000 C CNN
+F 4 "1276-1022-1-ND" H 1400 2350 60  0001 C CNN "Part No."
 	1    1400 2350
 	1    0    0    -1
@@
 F 0 "C11" H 1125 2450 50  0000 L CNN
 F 1 "1u" H 1125 2250 50  0000 L CNN
-F 2 "" H 1138 2200 50  0000 C CNN
+F 2 "Capacitors_SMD:C_0402" H 1138 2200 50  0001 C CNN
 F 3 "" H 1100 2350 50  0000 C CNN
+F 4 "1276-1448-1-ND" H 1100 2350 60  0001 C CNN "Part No."
 	1    1100 2350
 	1    0    0    -1
@@
 $EndComp
 Text Label 7150 2200 0    50   ~ 0
-USB_D+_R
+USB_D_R+
 Text Label 7150 2000 0    50   ~ 0
-USB_D-_R
+USB_D_R-
 $Comp
 L R R10
@@
 F 0 "R10" V 7830 2000 50  0000 C CNN
 F 1 "0" V 7750 2000 50  0000 C CNN
-F 2 "" V 7680 2000 50  0000 C CNN
+F 2 "Resistors_SMD:R_0402" V 7680 2000 50  0001 C CNN
 F 3 "" H 7750 2000 50  0000 C CNN
 	1    7750 2000
@@
 F 0 "R11" V 7830 2200 50  0000 C CNN
 F 1 "0" V 7750 2200 50  0000 C CNN
-F 2 "" V 7680 2200 50  0000 C CNN
+F 2 "Resistors_SMD:R_0402" V 7680 2200 50  0001 C CNN
 F 3 "" H 7750 2200 50  0000 C CNN
 	1    7750 2200
@@
 F 0 "C13" H 975 3100 50  0000 L CNN
 F 1 "C" H 975 2900 50  0000 L CNN
-F 2 "" H 988 2850 50  0000 C CNN
+F 2 "Capacitors_SMD:C_0402" H 988 2850 50  0001 C CNN
 F 3 "" H 950 3000 50  0000 C CNN
 	1    950  3000
@@
 F 0 "C14" H 975 3600 50  0000 L CNN
 F 1 "C" H 975 3400 50  0000 L CNN
-F 2 "" H 988 3350 50  0000 C CNN
+F 2 "Capacitors_SMD:C_0402" H 988 3350 50  0001 C CNN
 F 3 "" H 950 3500 50  0000 C CNN
 	1    950  3500
@@
 F 0 "P2" H 1200 5000 50  0000 C CNN
 F 1 "SWD" V 1300 4750 50  0000 C CNN
-F 2 "" H 1200 4750 50  0000 C CNN
+F 2 "" H 1200 4750 50  0001 C CNN
 F 3 "" H 1200 4750 50  0000 C CNN
 	1    1200 4750
@@
 F 0 "C15" H 725 6550 50  0000 L CNN
 F 1 "1u" H 725 6350 50  0000 L CNN
-F 2 "" H 738 6300 50  0000 C CNN
+F 2 "Capacitors_SMD:C_0402" H 738 6300 50  0001 C CNN
 F 3 "" H 700 6450 50  0000 C CNN
+F 4 "1276-1448-1-ND" H 700 6450 60  0001 C CNN "Part No."
 	1    700  6450
 	1    0    0    -1
@@
 F 0 "C16" H 925 6550 50  0000 L CNN
 F 1 "0.1u" H 925 6350 50  0000 L CNN
-F 2 "" H 938 6300 50  0000 C CNN
+F 2 "Capacitors_SMD:C_0402" H 938 6300 50  0001 C CNN
 F 3 "" H 900 6450 50  0000 C CNN
+F 4 "1276-1022-1-ND" H 900 6450 60  0001 C CNN "Part No."
 	1    900  6450
 	1    0    0    -1
@@
 F 0 "C17" H 1325 6550 50  0000 L CNN
 F 1 "0.1u" H 1325 6350 50  0000 L CNN
-F 2 "" H 1338 6300 50  0000 C CNN
+F 2 "Capacitors_SMD:C_0402" H 1338 6300 50  0001 C CNN
 F 3 "" H 1300 6450 50  0000 C CNN
+F 4 "1276-1022-1-ND" H 1300 6450 60  0001 C CNN "Part No."
 	1    1300 6450
 	1    0    0    -1
@@
 F 0 "C18" H 1525 7150 50  0000 L CNN
 F 1 "0.1u" H 1525 6950 50  0000 L CNN
-F 2 "" H 1538 6900 50  0000 C CNN
+F 2 "Capacitors_SMD:C_0402" H 1538 6900 50  0001 C CNN
 F 3 "" H 1500 7050 50  0000 C CNN
+F 4 "1276-1022-1-ND" H 1500 7050 60  0001 C CNN "Part No."
 	1    1500 7050
 	1    0    0    -1
@@
 F 0 "R16" V 9180 5750 50  0000 C CNN
 F 1 "4.7K" V 9100 5750 50  0000 C CNN
-F 2 "" V 9030 5750 50  0000 C CNN
+F 2 "Resistors_SMD:R_0402" V 9030 5750 50  0001 C CNN
 F 3 "" H 9100 5750 50  0000 C CNN
 	1    9100 5750
@@
 F 0 "R15" V 8980 5750 50  0000 C CNN
 F 1 "4.7K" V 8900 5750 50  0000 C CNN
-F 2 "" V 8830 5750 50  0000 C CNN
+F 2 "Resistors_SMD:R_0402" V 8830 5750 50  0001 C CNN
 F 3 "" H 8900 5750 50  0000 C CNN
 	1    8900 5750
@@
 F 0 "R17" V 3080 5850 50  0000 C CNN
 F 1 "10K" V 3000 5850 50  0000 C CNN
-F 2 "" V 2930 5850 50  0000 C CNN
+F 2 "Resistors_SMD:R_0402" V 2930 5850 50  0001 C CNN
 F 3 "" H 3000 5850 50  0000 C CNN
 	1    3000 5850
@@
 F 0 "R14" V 780 5750 50  0000 C CNN
 F 1 "0" V 700 5750 50  0000 C CNN
-F 2 "" V 630 5750 50  0000 C CNN
+F 2 "Resistors_SMD:R_0402" V 630 5750 50  0001 C CNN
 F 3 "" H 700 5750 50  0000 C CNN
 	1    700  5750
@@
 F 0 "R9" V 780 950 50  0000 C CNN
 F 1 "0" V 700 950 50  0000 C CNN
-F 2 "" V 630 950 50  0000 C CNN
+F 2 "Resistors_SMD:R_0402" V 630 950 50  0001 C CNN
 F 3 "" H 700 950 50  0000 C CNN
 	1    700  950
 	1    0    0    -1
 $EndComp
-Text Label 1100 900  0    50   ~ 0
-STM32_VDD
 Text Notes 900  700  0    50   ~ 0
 This resistor for current measurement if necessary
@@
 F 0 "R12" V 9080 3050 50  0000 C CNN
 F 1 "10K" V 9000 3050 50  0000 C CNN
-F 2 "" V 8930 3050 50  0000 C CNN
+F 2 "Resistors_SMD:R_0402" V 8930 3050 50  0001 C CNN
 F 3 "" H 9000 3050 50  0000 C CNN
 	1    9000 3050
@@
 F 0 "L2" H 700 1750 50  0000 C CNN
 F 1 "10u" H 700 1600 50  0000 C CNN
-F 2 "" H 700 1650 50  0000 C CNN
+F 2 "Resistors_SMD:R_0603" H 700 1650 50  0001 C CNN
 F 3 "" H 700 1650 50  0000 C CNN
+F 4 "445-6755-1-ND" H 700 1650 60  0001 C CNN "Part No."
 	1    700  1650
 	0    -1   -1   0
@@
 F 0 "R18" V 6130 6100 50  0000 C CNN
 F 1 "1K" V 6050 6100 50  0000 C CNN
-F 2 "" V 5980 6100 50  0000 C CNN
+F 2 "Resistors_SMD:R_0402" V 5980 6100 50  0001 C CNN
 F 3 "" H 6050 6100 50  0000 C CNN
 	1    6050 6100
@@
 P 6700 5200
 F 0 "D4" H 6650 5280 50  0000 L CNN
-F 1 "D_Small" H 6550 5120 50  0000 L CNN
-F 2 "" V 6700 5200 50  0000 C CNN
+F 1 "RB521S30T5G" H 6550 5120 50  0000 L CNN
+F 2 "Diodes_SMD:SOD-523" V 6700 5200 50  0001 C CNN
 F 3 "" V 6700 5200 50  0000 C CNN
+F 4 "B521S30T5GOSCT-ND" H 6700 5200 60  0001 C CNN "Part No."
 	1    6700 5200
 	0    1    1    0
@@
 F 0 "R13" V 6780 5650 50  0000 C CNN
 F 1 "R" V 6700 5650 50  0000 C CNN
-F 2 "" V 6630 5650 50  0000 C CNN
+F 2 "Resistors_SMD:R_0402" V 6630 5650 50  0001 C CNN
 F 3 "" H 6700 5650 50  0000 C CNN
 	1    6700 5650
@@
 Text Notes 7900 4500 0    50   ~ 0
 Also note that the button pin numbers\ndo not intersect any other interrupted\npin numbers so they can be waking\ninterrupts.
+Wire Wire Line
+	700  5550 600  5550
+Wire Wire Line
+	600  5550 600  5950
+Wire Wire Line
+	600  5950 700  5950
+Connection ~ 700  5950
+Connection ~ 700  5550
+Wire Wire Line
+	700  750  550  750
+Wire Wire Line
+	550  750  550  1150
+Wire Wire Line
+	550  1150 700  1150
+Connection ~ 700  1150
+Connection ~ 700  750
 $EndSCHEMATC

Commit message: Finished initial placement of all components
Got rid of several pullup resistors and unnecessary components.
Parts:
- removed L2: 10u, Resistors_SMD:R_0603, symbol INDUCTOR_SMALL
- removed R14, R9: 0, Resistors_SMD:R_0402, symbol R
- removed R17: 10K, Resistors_SMD:R_0402, symbol R
Connections:
- net STM32_VDDA is gone; now on net +3V3: C11.1, C12.1, U3.9 (VDDA)
- net STM32_OSC32_IN renamed STM32_OSC32+
- net STM32_OSC32_OUT renamed STM32_OSC32-
Other:
- note added: "Keep this pullup to keep\nthe lights off when the\nprocessor shuts down."
- note added: "Pullup provided by STM32"
- note removed: "This resistor for current\nmeasurement if needed"

Commit message: Routed most of the board, except buttons and interrupts
Parts:
- removed R12: 10K, Resistors_SMD:R_0402, symbol R
Connections:
- net STM32_OSC32+: now also Y1.2; no longer Y1.1
- net STM32_OSC32-: now also Y1.1; no longer Y1.2
Other:
- note added: "No pullup on led enable:\n1. When the microcontroller is off, it could float\nactive. However, the microcontroller's LED\noutputs are Hi-Z, so no current flows.\n2. When the microcontroller is on, it will be\nconfigured for open drain mode or normal GPIO\nmode. All is well."
- note removed: "Keep this pullup to keep\nthe lights off when the\nprocessor shuts down."
Changed lines of the file:
@@
 F 4 "370-1057-1-ND" H 1300 3250 60  0001 C CNN "Part No."
 	1    1300 3250
-	0    1    1    0
+	0    -1   -1   0
 $EndComp
 $Comp
@@
 Text HLabel 9100 3300 2    50   Input ~ 0
 ~LED_C_EN
-$Comp
-L R R12
-U 1 1 5801C130
-P 9000 3050
-F 0 "R12" V 9080 3050 50  0000 C CNN
-F 1 "10K" V 9000 3050 50  0000 C CNN
-F 2 "Resistors_SMD:R_0402" V 8930 3050 50  0001 C CNN
-F 3 "" H 9000 3050 50  0000 C CNN
-	1    9000 3050
-	1    0    0    -1
-$EndComp
-$Comp
-L +3.3V #PWR029
-U 1 1 5801C3D8
-P 9000 2800
-F 0 "#PWR029" H 9000 2650 50  0001 C CNN
-F 1 "+3.3V" H 9000 2940 50  0000 C CNN
-F 2 "" H 9000 2800 50  0000 C CNN
-F 3 "" H 9000 2800 50  0000 C CNN
-	1    9000 2800
-	1    0    0    -1
-$EndComp
 Text Notes 7900 4100 0    50   ~ 0
 Button pins chosen because of TSC\ngroup. Maybe in the future we can\nuse capacitive sensors and make a\nwaterproof case (would require\nsacrificing a button for Cs)
@@
 Text Notes 7900 4500 0    50   ~ 0
 Also note that the button pin numbers\ndo not intersect any other interrupted\npin numbers so they can be waking\ninterrupts.
-Text Notes 9200 3050 0    50   ~ 0
-Keep this pullup to keep\nthe lights off when the\nprocessor shuts down.
+Text Notes 8650 3200 0    50   ~ 0
+No pullup on led enable:\n1. When the microcontroller is off, it could float\nactive. However, the microcontroller's LED\noutputs are Hi-Z, so no current flows.\n2. When the microcontroller is on, it will be\nconfigured for open drain mode or normal GPIO\nmode. All is well.
 Text Notes 3150 5900 0    50   ~ 0
 Pullup provided by STM32
@@
 	5500 3300 9100 3300
 Wire Wire Line
-	9000 3200 9000 3300
-Connection ~ 9000 3300
-Wire Wire Line
-	9000 2800 9000 2900
-Wire Wire Line
 	6100 2800 5500 2800

Commit message: Selected programming header
Only one non-connected trace left. And I don't know where it is...
Parts:
- P2: footprint (none) -> simple-led-watch:JST-SH-4; Part No. (none) -> 455-1790-1-ND
Connections:
- net STM32_RESET: now also P2.2 (P2); no longer P2.4 (P4)
- net SWCLK: now also P2.3 (P3); no longer P2.2 (P2)
- net SWDIO: now also P2.4 (P4); no longer P2.3 (P3)
Other:
- note added: "Housing: 455-1379-ND\nCrimp socket: 455-1561-1-ND"
Changed lines of the file:
@@
 F 0 "P2" H 1200 5000 50  0000 C CNN
 F 1 "SWD" V 1300 4750 50  0000 C CNN
-F 2 "" H 1200 4750 50  0001 C CNN
+F 2 "simple-led-watch:JST-SH-4" H 1200 4750 50  0001 C CNN
 F 3 "" H 1200 4750 50  0000 C CNN
+F 4 "455-1790-1-ND" H 1200 4750 60  0001 C CNN "Part No."
 	1    1200 4750
 	-1   0    0    1
@@
 Text Label 6300 2300 0    50   ~ 0
 SWCLK
+Text Label 1800 4700 0    50   ~ 0
+SWCLK
+Text Label 1800 4600 0    50   ~ 0
+SWDIO
 Text Label 1800 4800 0    50   ~ 0
-SWCLK
-Text Label 1800 4700 0    50   ~ 0
-SWDIO
-Text Label 1800 4600 0    50   ~ 0
 STM32_RESET
 Text Label 2600 4000 2    50   ~ 0
@@
 $EndComp
 $Comp
-L +3.3V #PWR030
+L +3.3V #PWR029
 U 1 1 58024910
 P 6700 4850
-F 0 "#PWR030" H 6700 4700 50  0001 C CNN
+F 0 "#PWR029" H 6700 4700 50  0001 C CNN
 F 1 "+3.3V" H 6700 4990 50  0000 C CNN
 F 2 "" H 6700 4850 50  0000 C CNN
@@
 $EndComp
 $Comp
-L GND #PWR031
+L GND #PWR030
 U 1 1 58024E53
 P 6700 6400
-F 0 "#PWR031" H 6700 6150 50  0001 C CNN
+F 0 "#PWR030" H 6700 6150 50  0001 C CNN
 F 1 "GND" H 6700 6250 50  0000 C CNN
 F 2 "" H 6700 6400 50  0000 C CNN
@@
 	5500 2200 6300 2200
 Wire Wire Line
-	1400 4800 1800 4800
-Wire Wire Line
-	1800 4700 1400 4700
+	1400 4700 1800 4700
 Wire Wire Line
 	1800 4600 1400 4600
+Wire Wire Line
+	1800 4800 1400 4800
 Wire Wire Line
 	2600 4000 2900 4000
@@
 Wire Wire Line
 	6700 5800 6700 5900
+Text Notes 800  4500 0    50   ~ 0
+Housing: 455-1379-ND\nCrimp socket: 455-1561-1-ND
 $EndSCHEMATC

Commit message: Placed parts for round two
I'm pretty sure I can do it better
Connections:
- net STM32_OSC32+: now also Y1.1; no longer Y1.2
- net STM32_OSC32-: now also Y1.2; no longer Y1.1
Changed lines of the file:
@@
 F 4 "370-1057-1-ND" H 1300 3250 60  0001 C CNN "Part No."
 	1    1300 3250
-	0    -1   -1   0
+	0    1    1    0
 $EndComp
 $Comp

Commit message: Upgrade to latest kicad, add some measurements
Parts:
- D4: Part No. B521S30T5GOSCT-ND -> RB521S30T5GOSCT-ND
Changed lines of the file:
@@
 EESchema Schematic File Version 2
+LIBS:simple-led-watch-rescue
 LIBS:power
 LIBS:device
@@
 F 2 "Diodes_SMD:SOD-523" V 6700 5200 50  0001 C CNN
 F 3 "" V 6700 5200 50  0000 C CNN
-F 4 "B521S30T5GOSCT-ND" H 6700 5200 60  0001 C CNN "Part No."
+F 4 "RB521S30T5GOSCT-ND" H 6700 5200 60  0001 C CNN "Part No."
 	1    6700 5200
 	0    1    1    0
