File: kicad/control.sch (KiCad schematic (older format))
At the start: 25 parts, among them P2 SWD, Q2 MMBT3904, U3 STM32L052CxTx, U4 MMA8652FC, Y1 32.767KHz

Commit message: Checked layout and reference designs, swapped crystal and RGB LED
ST has a list of suggested crystals which are known to work with the
STM32L0 family. I selected one of those and it is significantly
smaller in all dimensions.

The RGB LED had too high of a green voltage. I swapped it out for a
slightly more expensive one with the same footprint that had startlingly
low green and blue forward voltages.

For layout changes:
- Fixed regulator footprint silkscreen
- Fixed regulator layout to be closer to reference design
- Fixed inductor silkscreen
- Moved accelerometer downward to accomodate capacitors above
- Fixed accelerometer layout to have no traces beneath
- Fixed accelerometer silkscreen
- Fixed LED silkscreen
- General small silkscreen edits, such as shifting text around

I've also chosen parts and values for all resistors and capacitors.
Parts:
- C13, C14: value C -> 8.2p; Part No. (none) -> 490-6256-1-ND
- R10, R11: Part No. (none) -> 311-0.0JRCT-ND
- R13: value R -> 0; Part No. (none) -> 311-0.0JRCT-ND
- R15, R16: Part No. (none) -> 311-4.7KLRCT-ND
- R18: Part No. (none) -> 311-10.0KLRCT-ND
- U3: value STM32L052CxTx -> STM32L052x8; symbol STM32L052CxTx -> STM32L052x8
- Y1: footprint simple-led-watch:XTAL-CPFB -> simple-led-watch:Crystal-Abracon-ABS07; Part No. 370-1057-1-ND -> 535-11937-1-ND
Other:
- note added: "R13 is just in case the buzzer\nis too loud. The datasheet\nimplies that it doesn't need any\ncurrent limiting."
Changed lines of the file:
@@
 F 2 "Resistors_SMD:R_0402" V 7680 2000 50  0001 C CNN
 F 3 "" H 7750 2000 50  0000 C CNN
+F 4 "311-0.0JRCT-ND" H 7750 2000 60  0001 C CNN "Part No."
 	1    7750 2000
 	0    -1   1    0
@@
 F 2 "Resistors_SMD:R_0402" V 7680 2200 50  0001 C CNN
 F 3 "" H 7750 2200 50  0000 C CNN
+F 4 "311-0.0JRCT-ND" H 7750 2200 60  0001 C CNN "Part No."
 	1    7750 2200
 	0    -1   1    0
@@
 F 0 "Y1" H 1300 3400 50  0000 C CNN
 F 1 "32.767KHz" H 1300 3100 50  0000 C CNN
-F 2 "simple-led-watch:XTAL-CPFB" H 1300 3250 50  0001 C CNN
+F 2 "simple-led-watch:Crystal-Abracon-ABS07" H 1300 3250 50  0001 C CNN
 F 3 "" H 1300 3250 50  0000 C CNN
-F 4 "370-1057-1-ND" H 1300 3250 60  0001 C CNN "Part No."
+F 4 "535-11937-1-ND" H 1300 3250 60  0001 C CNN "Part No."
 	1    1300 3250
 	0    1    1    0
@@
 P 950 3000
 F 0 "C13" H 975 3100 50  0000 L CNN
-F 1 "C" H 975 2900 50  0000 L CNN
+F 1 "8.2p" H 975 2900 50  0000 L CNN
 F 2 "Capacitors_SMD:C_0402" H 988 2850 50  0001 C CNN
 F 3 "" H 950 3000 50  0000 C CNN
+F 4 "490-6256-1-ND" H 950 3000 60  0001 C CNN "Part No."
 	1    950  3000
 	0    1    1    0
@@
 P 950 3500
 F 0 "C14" H 975 3600 50  0000 L CNN
-F 1 "C" H 975 3400 50  0000 L CNN
+F 1 "8.2p" H 975 3400 50  0000 L CNN
 F 2 "Capacitors_SMD:C_0402" H 988 3350 50  0001 C CNN
 F 3 "" H 950 3500 50  0000 C CNN
+F 4 "490-6256-1-ND" H 950 3500 60  0001 C CNN "Part No."
 	1    950  3500
 	0    1    1    0
@@
 F 2 "Resistors_SMD:R_0402" V 9030 5750 50  0001 C CNN
 F 3 "" H 9100 5750 50  0000 C CNN
+F 4 "311-4.7KLRCT-ND" H 9100 5750 60  0001 C CNN "Part No."
 	1    9100 5750
 	1    0    0    -1
@@
 F 2 "Resistors_SMD:R_0402" V 8830 5750 50  0001 C CNN
 F 3 "" H 8900 5750 50  0000 C CNN
+F 4 "311-4.7KLRCT-ND" H 8900 5750 60  0001 C CNN "Part No."
 	1    8900 5750
 	1    0    0    -1
@@
 F 2 "Resistors_SMD:R_0402" V 5980 6100 50  0001 C CNN
 F 3 "" H 6050 6100 50  0000 C CNN
+F 4 "311-10.0KLRCT-ND" H 6050 6100 60  0001 C CNN "Part No."
 	1    6050 6100
 	0    1    1    0
@@
 P 6700 5650
 F 0 "R13" V 6780 5650 50  0000 C CNN
-F 1 "R" V 6700 5650 50  0000 C CNN
+F 1 "0" V 6700 5650 50  0000 C CNN
 F 2 "Resistors_SMD:R_0402" V 6630 5650 50  0001 C CNN
 F 3 "" H 6700 5650 50  0000 C CNN
+F 4 "311-0.0JRCT-ND" H 6700 5650 60  0001 C CNN "Part No."
 	1    6700 5650
 	1    0    0    -1
@@
 Housing: 455-1379-ND\nCrimp socket: 455-1561-1-ND
 $Comp
-L STM32L052CxTx U3
+L STM32L052x8 U3
 U 1 1 57FCAB90
 P 4200 2500
 F 0 "U3" H 4200 750 50  0000 C CNN
-F 1 "STM32L052CxTx" H 4200 4250 50  0000 C CNN
+F 1 "STM32L052x8" H 4200 4250 50  0000 C CNN
 F 2 "Housings_QFP:LQFP-48_7x7mm_Pitch0.5mm" H 4200 2900 50  0001 C CNN
 F 3 "" H 4200 2900 50  0001 C CNN
@@
 $EndComp
 NoConn ~ 5500 1600
+Text Notes 7000 6000 0    50   ~ 0
+R13 is just in case the buzzer\nis too loud. The datasheet\nimplies that it doesn't need any\ncurrent limiting.
 $EndSCHEMATC
