File: kicad/power-supply.sch (KiCad schematic (older format))
At the start: 22 parts, among them P1 BATTERY, Q1 Q_NPN_EBC, U1 MCP73832, U2 TPS62736

Commit message: Added footprints for most major components
We are missing almost all passives
Parts:
- removed Q1: Q_NPN_EBC, symbol Q_NPN_EBC
- added Q1: MMBT3904, TO_SOT_Packages_SMD:SOT-23, symbol Q_NPN_BEC
- L1: footprint (none) -> simple-led-watch:SMD_1008
- P1: footprint (none) -> simple-led-watch:JST-ACH-2PIN; Part No. (none) -> 455-2202-1-ND
- U1: footprint (none) -> TO_SOT_Packages_SMD:SOT-23-5
- U2: footprint (none) -> simple-led-watch:14-VQFN
Changed lines of the file:
@@
 F 0 "U2" H 7400 4100 60  0000 C CNN
 F 1 "TPS62736" H 7400 5400 60  0000 C CNN
-F 2 "" H 7400 4900 60  0001 C CNN
+F 2 "simple-led-watch:14-VQFN" H 7400 4900 60  0001 C CNN
 F 3 "" H 7400 4900 60  0001 C CNN
 F 4 "296-43622-1-ND" H 7400 4700 60  0001 C CNN "Part No."
@@
 F 0 "U1" H 2800 1150 60  0000 C CNN
 F 1 "MCP73832" H 2800 1850 60  0000 C CNN
-F 2 "" H 2800 1500 60  0001 C CNN
+F 2 "TO_SOT_Packages_SMD:SOT-23-5" H 2800 1500 60  0001 C CNN
 F 3 "" H 2800 1500 60  0001 C CNN
 F 4 "MCP73832T-2DCI/OTCT-ND" H 2800 1500 60  0001 C CNN "Part No."
@@
 F 0 "P1" H 4800 1500 50  0000 C CNN
 F 1 "BATTERY" V 4900 1350 50  0000 C CNN
-F 2 "" H 4800 1350 50  0000 C CNN
+F 2 "simple-led-watch:JST-ACH-2PIN" H 4800 1350 50  0001 C CNN
 F 3 "" H 4800 1350 50  0000 C CNN
+F 4 "455-2202-1-ND" H 4800 1350 60  0001 C CNN "Part No."
 	1    4800 1350
 	1    0    0    -1
@@
 $EndComp
 $Comp
-L GND #PWR4
+L GND #PWR01
 U 1 1 57FA8D3B
 P 3700 2100
-F 0 "#PWR4" H 3700 1850 50  0001 C CNN
+F 0 "#PWR01" H 3700 1850 50  0001 C CNN
 F 1 "GND" H 3700 1950 50  0000 C CNN
 F 2 "" H 3700 2100 50  0000 C CNN
@@
 $EndComp
 $Comp
-L GND #PWR1
+L GND #PWR02
 U 1 1 57FA90ED
 P 4500 1500
-F 0 "#PWR1" H 4500 1250 50  0001 C CNN
+F 0 "#PWR02" H 4500 1250 50  0001 C CNN
 F 1 "GND" H 4500 1350 50  0000 C CNN
 F 2 "" H 4500 1500 50  0000 C CNN
@@
 $EndComp
 $Comp
-L GND #PWR5
+L GND #PWR03
 U 1 1 57FA9276
 P 4000 2100
-F 0 "#PWR5" H 4000 1850 50  0001 C CNN
+F 0 "#PWR03" H 4000 1850 50  0001 C CNN
 F 1 "GND" H 4000 1950 50  0000 C CNN
 F 2 "" H 4000 2100 50  0000 C CNN
@@
 F 0 "L1" H 8550 4300 50  0000 C CNN
 F 1 "10u" H 8550 4150 50  0000 C CNN
-F 2 "" H 8550 4200 50  0000 C CNN
+F 2 "simple-led-watch:SMD_1008" H 8550 4200 50  0001 C CNN
 F 3 "" H 8550 4200 50  0000 C CNN
 F 4 "490-10563-1-ND" H 8550 4200 60  0001 C CNN "Part No."
@@
 $EndComp
 $Comp
-L GND #PWR2
+L GND #PWR04
 U 1 1 57FA9B89
 P 1600 1800
-F 0 "#PWR2" H 1600 1550 50  0001 C CNN
+F 0 "#PWR04" H 1600 1550 50  0001 C CNN
 F 1 "GND" H 1600 1650 50  0000 C CNN
 F 2 "" H 1600 1800 50  0000 C CNN
@@
 $EndComp
 $Comp
-L GND #PWR3
+L GND #PWR05
 U 1 1 57FA9BB9
 P 1850 1800
-F 0 "#PWR3" H 1850 1550 50  0001 C CNN
+F 0 "#PWR05" H 1850 1550 50  0001 C CNN
 F 1 "GND" H 1850 1650 50  0000 C CNN
 F 2 "" H 1850 1800 50  0000 C CNN
@@
 $EndComp
 $Comp
-L GND #PWR11
+L GND #PWR06
 U 1 1 57FB0678
 P 8200 5300
-F 0 "#PWR11" H 8200 5050 50  0001 C CNN
+F 0 "#PWR06" H 8200 5050 50  0001 C CNN
 F 1 "GND" H 8200 5150 50  0000 C CNN
 F 2 "" H 8200 5300 50  0000 C CNN
@@
 Low eakage diode to prevent backpowering\nwhen USB isn't plugged in
 $Comp
-L GND #PWR12
+L GND #PWR07
 U 1 1 57FB19E3
 P 9000 5300
-F 0 "#PWR12" H 9000 5050 50  0001 C CNN
+F 0 "#PWR07" H 9000 5050 50  0001 C CNN
 F 1 "GND" H 9000 5150 50  0000 C CNN
 F 2 "" H 9000 5300 50  0000 C CNN
@@
 $EndComp
 $Comp
-L GND #PWR13
+L GND #PWR08
 U 1 1 57FC59D4
 P 9900 5300
-F 0 "#PWR13" H 9900 5050 50  0001 C CNN
+F 0 "#PWR08" H 9900 5050 50  0001 C CNN
 F 1 "GND" H 9900 5150 50  0000 C CNN
 F 2 "" H 9900 5300 50  0000 C CNN
@@
 $EndComp
 $Comp
-L +3.3V #PWR9
+L +3.3V #PWR09
 U 1 1 57FC5A4F
 P 9900 4100
-F 0 "#PWR9" H 9900 3950 50  0001 C CNN
+F 0 "#PWR09" H 9900 3950 50  0001 C CNN
 F 1 "+3.3V" H 9900 4240 50  0000 C CNN
 F 2 "" H 9900 4100 50  0000 C CNN
@@
 $EndComp
 $Comp
-L GND #PWR14
+L GND #PWR010
 U 1 1 57FC5D97
 P 5300 5450
-F 0 "#PWR14" H 5300 5200 50  0001 C CNN
+F 0 "#PWR010" H 5300 5200 50  0001 C CNN
 F 1 "GND" H 5300 5300 50  0000 C CNN
 F 2 "" H 5300 5450 50  0000 C CNN
@@
 $EndComp
 $Comp
-L GND #PWR15
+L GND #PWR011
 U 1 1 57FC6553
 P 5700 6000
-F 0 "#PWR15" H 5700 5750 50  0001 C CNN
+F 0 "#PWR011" H 5700 5750 50  0001 C CNN
 F 1 "GND" H 5700 5850 50  0000 C CNN
 F 2 "" H 5700 6000 50  0000 C CNN
@@
 $EndComp
 $Comp
-L GND #PWR16
+L GND #PWR012
 U 1 1 57FC6D09
 P 6100 6000
-F 0 "#PWR16" H 6100 5750 50  0001 C CNN
+F 0 "#PWR012" H 6100 5750 50  0001 C CNN
 F 1 "GND" H 6100 5850 50  0000 C CNN
 F 2 "" H 6100 6000 50  0000 C CNN
@@
 $EndComp
 $Comp
-L GND #PWR10
+L GND #PWR013
 U 1 1 57FC72B8
 P 6300 4700
-F 0 "#PWR10" H 6300 4450 50  0001 C CNN
+F 0 "#PWR013" H 6300 4450 50  0001 C CNN
 F 1 "GND" H 6300 4550 50  0000 C CNN
 F 2 "" H 6300 4700 50  0000 C CNN
@@
 $EndComp
 $Comp
-L +3.3V #PWR6
+L +3.3V #PWR014
 U 1 1 57FC7C6B
 P 6300 2200
-F 0 "#PWR6" H 6300 2050 50  0001 C CNN
+F 0 "#PWR014" H 6300 2050 50  0001 C CNN
 F 1 "+3.3V" H 6300 2340 50  0000 C CNN
 F 2 "" H 6300 2200 50  0000 C CNN
@@
 CHG_STAT
 $Comp
-L +3.3V #PWR7
+L +3.3V #PWR015
 U 1 1 57FC80A3
 P 8200 2200
-F 0 "#PWR7" H 8200 2050 50  0001 C CNN
+F 0 "#PWR015" H 8200 2050 50  0001 C CNN
 F 1 "+3.3V" H 8200 2340 50  0000 C CNN
 F 2 "" H 8200 2200 50  0000 C CNN
@@
 F 3 "" H 8200 2450 50  0000 C CNN
 	1    8200 2450
-	1    0    0    -1
-$EndComp
-$Comp
-L Q_NPN_EBC Q1
-U 1 1 57FC81BB
-P 3000 2600
-F 0 "Q1" H 3300 2650 50  0000 R CNN
-F 1 "Q_NPN_EBC" H 3600 2550 50  0000 R CNN
-F 2 "" H 3200 2700 50  0000 C CNN
-F 3 "" H 3000 2600 50  0000 C CNN
-	1    3000 2600
 	1    0    0    -1
 $EndComp
@@
 $EndComp
 $Comp
-L GND #PWR8
+L GND #PWR016
 U 1 1 57FC84EA
 P 3100 2900
-F 0 "#PWR8" H 3100 2650 50  0001 C CNN
+F 0 "#PWR016" H 3100 2650 50  0001 C CNN
 F 1 "GND" H 3100 2750 50  0000 C CNN
 F 2 "" H 3100 2900 50  0000 C CNN
@@
 Text Notes 4450 3150 0    50   ~ 0
 Voltage drop is critical for this one. When\nconducting, we are under battery power.
+$Comp
+L Q_NPN_BEC Q1
+U 1 1 58030BFE
+P 3000 2600
+F 0 "Q1" H 3300 2650 50  0000 R CNN
+F 1 "MMBT3904" H 3600 2550 50  0000 R CNN
+F 2 "TO_SOT_Packages_SMD:SOT-23" H 3200 2700 50  0001 C CNN
+F 3 "" H 3000 2600 50  0000 C CNN
+F 4 "MMBT3904FSCT-ND" H 3000 2600 60  0001 C CNN "Part No."
+	1    3000 2600
+	1    0    0    -1
+$EndComp
 $EndSCHEMATC

Commit message: Completed initial placement of major components
The passives are causing trouble. We need to eliminate every pullup
possible.
Parts:
- C1: footprint (none) -> Capacitors_SMD:C_0402; Part No. (none) -> 1276-1448-1-ND
- C2: footprint (none) -> Capacitors_SMD:C_0402; Part No. (none) -> 1276-1022-1-ND
- C3, C5: footprint (none) -> Capacitors_SMD:C_0402; Part No. (none) -> 1276-6819-1-ND
- C4, C6: footprint (none) -> Capacitors_SMD:C_0603; Part No. (none) -> 1276-6504-1-ND
- D1: value D_Small -> CDSU101A; footprint (none) -> Diodes_SMD:SOD-523; Part No. (none) -> 641-1002-1-ND
- D2: value D_Schottky_Small -> RB521S30T5G; footprint (none) -> Diodes_SMD:SOD-523; Part No. (none) -> RB521S30T5GOSCT-ND
- R1, R2, R3, R4, R5, R6, R7, R8: footprint (none) -> Resistors_SMD:R_0402
Connections:
- net +3V3: now also R3.1
- net +3.3V_REG_SRC: now reaches C4.1, C5.1, D1.1 (K), D2.1 (K), U2.1 (IN), U2.6 (EN2)
- net +3.3V_REG_SW: now reaches L1.1, U2.13 (SW)
- net +3.3V_REG_VRDIV: now reaches R5.1, R6.1, U2.7 (VRDIV)
- net +3.3V_REG_VOK_SET: now reaches R6.2, R8.1, U2.8 (VIN_OK_SET)
- net +3.3V_REG_VOUT_SET: now reaches R5.2, R7.1, U2.9 (VOUT_SET)
Other:
- note added: "Voltage drop is critical for this one. When\nconducting, we are under battery power.\nAlso remember that current will fluctuate\ndrastically when the lights turn on."
- note removed: "Voltage drop is critical for this one. When\nconducting, we are under battery power."
Changed lines of the file:
@@
 F 0 "R1" V 3780 1750 50  0000 C CNN
 F 1 "20K" V 3700 1750 50  0000 C CNN
-F 2 "" V 3630 1750 50  0000 C CNN
+F 2 "Resistors_SMD:R_0402" V 3630 1750 50  0001 C CNN
 F 3 "" H 3700 1750 50  0000 C CNN
 	1    3700 1750
@@
 F 0 "C3" H 4025 1650 50  0000 L CNN
 F 1 "4.7u" H 4025 1450 50  0000 L CNN
-F 2 "" H 4038 1400 50  0000 C CNN
+F 2 "Capacitors_SMD:C_0402" H 4038 1400 50  0001 C CNN
 F 3 "" H 4000 1550 50  0000 C CNN
+F 4 "1276-6819-1-ND" H 4000 1550 60  0001 C CNN "Part No."
 	1    4000 1550
 	1    0    0    -1
@@
 F 0 "C5" H 5625 4650 50  0000 L CNN
 F 1 "4.7u" H 5625 4450 50  0000 L CNN
-F 2 "" H 5638 4400 50  0000 C CNN
+F 2 "Capacitors_SMD:C_0402" H 5638 4400 50  0001 C CNN
 F 3 "" H 5600 4550 50  0000 C CNN
+F 4 "1276-6819-1-ND" H 5600 4550 60  0001 C CNN "Part No."
 	1    5600 4550
 	1    0    0    -1
@@
 F 0 "C6" H 9025 4650 50  0000 L CNN
 F 1 "22u" H 9025 4450 50  0000 L CNN
-F 2 "" H 9038 4400 50  0000 C CNN
+F 2 "Capacitors_SMD:C_0603" H 9038 4400 50  0001 C CNN
 F 3 "" H 9000 4550 50  0000 C CNN
+F 4 "1276-6504-1-ND" H 9000 4550 60  0001 C CNN "Part No."
 	1    9000 4550
 	1    0    0    -1
@@
 F 0 "C1" H 1625 1650 50  0000 L CNN
 F 1 "1u" H 1625 1450 50  0000 L CNN
-F 2 "" H 1638 1400 50  0000 C CNN
+F 2 "Capacitors_SMD:C_0402" H 1638 1400 50  0001 C CNN
 F 3 "" H 1600 1550 50  0000 C CNN
+F 4 "1276-1448-1-ND" H 1600 1550 60  0001 C CNN "Part No."
 	1    1600 1550
 	1    0    0    -1
@@
 F 0 "C2" H 1875 1650 50  0000 L CNN
 F 1 "0.1u" H 1875 1450 50  0000 L CNN
-F 2 "" H 1888 1400 50  0000 C CNN
+F 2 "Capacitors_SMD:C_0402" H 1888 1400 50  0001 C CNN
 F 3 "" H 1850 1550 50  0000 C CNN
+F 4 "1276-1022-1-ND" H 1850 1550 60  0001 C CNN "Part No."
 	1    1850 1550
 	1    0    0    -1
@@
 F 0 "C4" H 5325 4650 50  0000 L CNN
 F 1 "22u" H 5325 4450 50  0000 L CNN
-F 2 "" H 5338 4400 50  0000 C CNN
+F 2 "Capacitors_SMD:C_0603" H 5338 4400 50  0001 C CNN
 F 3 "" H 5300 4550 50  0000 C CNN
+F 4 "1276-6504-1-ND" H 5300 4550 60  0001 C CNN "Part No."
 	1    5300 4550
 	1    0    0    -1
@@
 P 2300 3100
 F 0 "D1" H 2250 3180 50  0000 L CNN
-F 1 "D_Small" H 2150 3020 50  0000 L CNN
-F 2 "" V 2300 3100 50  0000 C CNN
+F 1 "CDSU101A" H 2150 3020 50  0000 L CNN
+F 2 "Diodes_SMD:SOD-523" V 2300 3100 50  0001 C CNN
 F 3 "" V 2300 3100 50  0000 C CNN
+F 4 "641-1002-1-ND" H 2300 3100 60  0001 C CNN "Part No."
 	1    2300 3100
 	0    -1   -1   0
@@
 P 4250 3100
 F 0 "D2" H 4200 3180 50  0000 L CNN
-F 1 "D_Schottky_Small" H 3970 3020 50  0000 L CNN
-F 2 "" V 4250 3100 50  0000 C CNN
+F 1 "RB521S30T5G" H 3970 3020 50  0000 L CNN
+F 2 "Diodes_SMD:SOD-523" V 4250 3100 50  0001 C CNN
 F 3 "" V 4250 3100 50  0000 C CNN
+F 4 "RB521S30T5GOSCT-ND" H 4250 3100 60  0001 C CNN "Part No."
 	1    4250 3100
 	0    -1   -1   0
@@
 F 0 "R5" V 5780 5250 50  0000 C CNN
 F 1 "6.3M" V 5700 5250 50  0000 C CNN
-F 2 "" V 5630 5250 50  0000 C CNN
+F 2 "Resistors_SMD:R_0402" V 5630 5250 50  0001 C CNN
 F 3 "" H 5700 5250 50  0000 C CNN
 	1    5700 5250
@@
 F 0 "R7" V 5780 5750 50  0000 C CNN
 F 1 "3.67M" V 5700 5750 50  0000 C CNN
-F 2 "" V 5630 5750 50  0000 C CNN
+F 2 "Resistors_SMD:R_0402" V 5630 5750 50  0001 C CNN
 F 3 "" H 5700 5750 50  0000 C CNN
 	1    5700 5750
@@
 F 0 "R6" V 6180 5250 50  0000 C CNN
 F 1 "6M" V 6100 5250 50  0000 C CNN
-F 2 "" V 6030 5250 50  0000 C CNN
+F 2 "Resistors_SMD:R_0402" V 6030 5250 50  0001 C CNN
 F 3 "" H 6100 5250 50  0000 C CNN
 	1    6100 5250
@@
 F 0 "R8" V 6180 5750 50  0000 C CNN
 F 1 "4M" V 6100 5750 50  0000 C CNN
-F 2 "" V 6030 5750 50  0000 C CNN
+F 2 "Resistors_SMD:R_0402" V 6030 5750 50  0001 C CNN
 F 3 "" H 6100 5750 50  0000 C CNN
 	1    6100 5750
@@
 F 0 "R2" V 6380 2450 50  0000 C CNN
 F 1 "10K" V 6300 2450 50  0000 C CNN
-F 2 "" V 6230 2450 50  0000 C CNN
+F 2 "Resistors_SMD:R_0402" V 6230 2450 50  0001 C CNN
 F 3 "" H 6300 2450 50  0000 C CNN
 	1    6300 2450
@@
 F 0 "R3" V 8280 2450 50  0000 C CNN
 F 1 "10K" V 8200 2450 50  0000 C CNN
-F 2 "" V 8130 2450 50  0000 C CNN
+F 2 "Resistors_SMD:R_0402" V 8130 2450 50  0001 C CNN
 F 3 "" H 8200 2450 50  0000 C CNN
 	1    8200 2450
@@
 F 0 "R4" V 2630 2600 50  0000 C CNN
 F 1 "1K" V 2550 2600 50  0000 C CNN
-F 2 "" V 2480 2600 50  0000 C CNN
+F 2 "Resistors_SMD:R_0402" V 2480 2600 50  0001 C CNN
 F 3 "" H 2550 2600 50  0000 C CNN
 	1    2550 2600
@@
 Connection ~ 8200 2700
 Text Notes 4450 3150 0    50   ~ 0
-Voltage drop is critical for this one. When\nconducting, we are under battery power.
+Voltage drop is critical for this one. When\nconducting, we are under battery power.\nAlso remember that current will fluctuate\ndrastically when the lights turn on.
 $Comp
 L Q_NPN_BEC Q1
@@
 	1    0    0    -1
 $EndComp
+Text Label 4500 4200 0    50   ~ 0
++3.3V_REG_SRC
+Text Label 5700 4900 0    50   ~ 0
++3.3V_REG_VRDIV
+Text Label 5900 5000 0    50   ~ 0
++3.3V_REG_VOUT_SET
+Text Label 6300 5100 0    50   ~ 0
++3.3V_REG_VOK_SET
+Text Label 8200 4200 1    50   ~ 0
++3.3V_REG_SW
+Wire Wire Line
+	8200 2300 8200 2200
 $EndSCHEMATC
